Commit message: Update to ROS Melodic

File: wrs_gazebo/mobile_dual_arm/urdf/mobile_dual_arm.xacro (robot description, xacro)
@@ -2,5 +2,5 @@
 <robot name="mobile_dual_arm" xmlns:xacro="http://www.ros.org/wiki/xacro">
   <xacro:include filename="$(find single_arm_description)/urdf/single_arm.xacro" />
-  <xacro:include filename="$(find Slide_rail)/urdf/Slide_rail.xacro" />
+  <xacro:include filename="$(find slide_rail)/urdf/slide_rail.xacro" />
   <xacro:include filename="$(find suction_urdf)/urdf/suction_urdf.xacro" />
   <!--xacro:include filename="$(find single_arm_description)/urdf/materials.xacro" /-->
@@ -105,5 +105,5 @@
   <transmission name="tran1_slide_R">
     <type>transmission_interface/SimpleTransmission</type>
-    <joint name="Slide_R">
+    <joint name="slide_R">
       <hardwareInterface>hardware_interface/PositionJointInterface</hardwareInterface>
     </joint>
@@ -115,5 +115,5 @@
   <transmission name="tran_slide_L">
     <type>transmission_interface/SimpleTransmission</type>
-    <joint name="Slide_L">
+    <joint name="slide_L">
       <hardwareInterface>hardware_interface/PositionJointInterface</hardwareInterface>
     </joint>

File: wrs_gazebo/slide_rail/urdf/slide_rail.urdf (robot description, URDF)
Before this commit: robot Slide_rail, 3 links, 2 joints
Links:
- link Arm_Base_L_Link: mass 0.2915148495066669 -> 0.0915148495066669; geometry collision mesh filename=package://slide_rail/meshes/Arm_Base_L_Link.STL; visual mesh filename=package://slide_rail/meshes/Arm_Base_L_Link.STL
- link Arm_Base_R_Link: mass 0.2915148495066668 -> 0.0915148495066668; geometry collision mesh filename=package://slide_rail/meshes/Arm_Base_R_Link.STL; visual mesh filename=package://slide_rail/meshes/Arm_Base_R_Link.STL
- link base_link: mass 1300.2157378026818 -> 13.2157378026818; geometry collision mesh filename=package://slide_rail/meshes/base_link.STL; visual mesh filename=package://slide_rail/meshes/base_link.STL
Joints:
- removed joint Slide_L
- removed joint Slide_R
- added joint slide_L: type prismatic, parent base_link, child Arm_Base_L_Link, origin xyz=-0.08 0.0925 0.88886 rpy=7.8352E-17 -1.301E-16 -3.8305E-16, axis 0 0 1, limit effort=0 velocity=0
- added joint slide_R: type prismatic, parent base_link, child Arm_Base_R_Link, origin xyz=-0.08 -0.0925 0.88886 rpy=-7.1169E-16 5.5825E-15 3.3307E-16, axis 0 0 1, limit effort=0 velocity=0

File: wrs_gazebo/slide_rail/urdf/slide_rail.xacro (robot description, xacro)
@@ -1,5 +1,5 @@
 <?xml version="1.0"?>
 <!-- Revolute-Revolute Manipulator -->
-<robot name="Slide_rail" xmlns:xacro="http://www.ros.org/wiki/xacro">
+<robot name="slide_rail" xmlns:xacro="http://www.ros.org/wiki/xacro">
   <link
     name="base_link">
@@ -9,5 +9,5 @@
         rpy="0 0 0" />
       <mass
-        value="13.2157378026818" />
+        value="1300.2157378026818" />
       <inertia
         ixx="1.5723643860749"
@@ -15,5 +15,5 @@
         ixz="-0.0259807481556023"
         iyy="1.56653528372694"
-        iyz="-0.0123413171800455"
+        iyz="-0.0223413171800455"
         izz="0.0334677964955424" />
     </inertial>
@@ -24,5 +24,5 @@
       <geometry>
         <mesh
-          filename="package://Slide_rail/meshes/base_link.STL" />
+          filename="package://slide_rail/meshes/base_link.STL" />
       </geometry>
       <material
@@ -38,5 +38,5 @@
       <geometry>
         <mesh
-          filename="package://Slide_rail/meshes/base_link.STL" />
+          filename="package://slide_rail/meshes/base_link.STL" />
       </geometry>
     </collision>
@@ -46,15 +46,15 @@
     <inertial>
       <origin
-        xyz="1.57200647357136E-05 0.022625966524659 -2.45861738434883E-06"
+        xyz="0 0.022625966524659 0"
         rpy="0 0 0" />
       <mass
-        value="0.0915148495066668" />
+        value="0.2915148495066668" />
       <inertia
-        ixx="8.99401518227245E-05"
+        ixx="1.50001518227245"
         ixy="6.65500499430702E-09"
         ixz="-5.17853701338548E-09"
-        iyy="0.000123418097290043"
+        iyy="1.50418097290043"
         iyz="-1.04084246775258E-09"
-        izz="3.58919292165612E-05" />
+        izz="0.029919292165612" />
     </inertial>
     <visual>
@@ -64,5 +64,5 @@
       <geometry>
         <mesh
-          filename="package://Slide_rail/meshes/Arm_Base_R_Link.STL" />
+          filename="package://slide_rail/meshes/Arm_Base_R_Link.STL" />
       </geometry>
       <material
@@ -78,14 +78,14 @@
       <geometry>
         <mesh
-          filename="package://Slide_rail/meshes/Arm_Base_R_Link.STL" />
+          filename="package://slide_rail/meshes/Arm_Base_R_Link.STL" />
       </geometry>
     </collision>
   </link>
   <joint
-    name="Slide_R"
+    name="slide_R"
     type="prismatic">
     <origin
       xyz="-0.08 -0.0925 0.88886"
-      rpy="-7.1169E-16 5.5825E-15 3.3307E-16" />
+      rpy="0 0 0" />
     <parent
       link="base_link" />
@@ -95,6 +95,8 @@
       xyz="0 0 1" />
     <limit
-      effort="0"
-      velocity="0" />
+      lower="-0.8"
+      upper="0"
+      effort="500"
+      velocity="100" />
   </joint>
   <link
@@ -102,15 +104,15 @@
     <inertial>
       <origin
-        xyz="-1.57200647414868E-05 -0.022625966524659 -2.45861739034403E-06"
+        xyz="0 -0.022625966524659 0"
         rpy="0 0 0" />
       <mass
-        value="0.0915148495066669" />
+        value="0.2915148495066669" />
       <inertia
-        ixx="8.99401518227246E-05"
+        ixx="1.501518227246"
         ixy="6.655004994278E-09"
         ixz="5.1785370134074E-09"
-        iyy="0.000123418097290043"
+        iyy="1.50418097290043"
         iyz="1.04084246778742E-09"
-        izz="3.58919292165613E-05" />
+        izz="0.29919292165613" />
     </inertial>
     <visual>
@@ -120,5 +122,5 @@
       <geometry>
         <mesh
-          filename="package://Slide_rail/meshes/Arm_Base_L_Link.STL" />
+          filename="package://slide_rail/meshes/Arm_Base_L_Link.STL" />
       </geometry>
       <material
@@ -134,14 +136,14 @@
       <geometry>
         <mesh
-          filename="package://Slide_rail/meshes/Arm_Base_L_Link.STL" />
+          filename="package://slide_rail/meshes/Arm_Base_L_Link.STL" />
       </geometry>
     </collision>
   </link>
   <joint
-    name="Slide_L"
+    name="slide_L"
     type="prismatic">
     <origin
       xyz="-0.08 0.0925 0.88886"
-      rpy="7.8352E-17 -1.301E-16 -3.8305E-16" />
+      rpy="0 0 0" />
     <parent
       link="base_link" />
@@ -151,6 +153,30 @@
       xyz="0 0 1" />
     <limit
-      effort="0"
-      velocity="0" />
+      lower="-0.8"
+      upper="0"
+      effort="500"
+      velocity="100" />
   </joint>
+<!--
+  <transmission name="tran1">
+    <type>transmission_interface/SimpleTransmission</type>
+    <joint name="slide_R">
+      <hardwareInterface>hardware_interface/PositionJointInterface</hardwareInterface>
+    </joint>
+    <actuator name="motor1">
+      <hardwareInterface>hardware_interface/PositionJointInterface</hardwareInterface>
+      <mechanicalReduction>1</mechanicalReduction>
+    </actuator>
+  </transmission>
+  <transmission name="tran2">
+    <type>transmission_interface/SimpleTransmission</type>
+    <joint name="slide_L">
+      <hardwareInterface>hardware_interface/PositionJointInterface</hardwareInterface>
+    </joint>
+    <actuator name="motor2">
+      <hardwareInterface>hardware_interface/PositionJointInterface</hardwareInterface>
+      <mechanicalReduction>1</mechanicalReduction>
+    </actuator>
+  </transmission>
+-->
 </robot>
