Commit message: Add Mir into Gazebo, Files not been Organized

File: wrs_gazebo/mobile_dual_arm/urdf/mobile_dual_arm.xacro (robot description, xacro)
@@ -1,11 +1,14 @@
 <?xml version="1.0"?>
 <robot name="mobile_dual_arm" xmlns:xacro="http://www.ros.org/wiki/xacro">
+  <xacro:include filename="$(find mir_description)/urdf/include/mir_100_v1.urdf.xacro" />
+  <!--<xacro:include filename="$(find mir_description)/urdf/include/common.gazebo.xacro" />-->
   <xacro:include filename="$(find single_arm_description)/urdf/single_arm.xacro" />
-  <xacro:include filename="$(find slide_rail)/urdf/slide_rail.xacro" />
+  <xacro:include filename="$(find timda_body)/urdf/timda_body.xacro" />
+  <!-- <xacro:include filename="$(find slide_rail)/urdf/slide_rail.xacro" /> -->
   <xacro:include filename="$(find suction_urdf)/urdf/suction_urdf.xacro" />
   <!--xacro:include filename="$(find single_arm_description)/urdf/materials.xacro" /-->
   <xacro:include filename="$(find mobile_dual_arm)/urdf/mobile_dual_arm.gazebo" />
-  <xacro:include filename="$(find mobile_table)/urdf/mobile_table.xacro" />
-  <link name="world"/>
+  <!--xacro:include filename="$(find mobile_table)/urdf/mobile_table.xacro" /-->
+  <!--<link name="world"/-->
   <!-- <joint name="fixed1" type="fixed">
     <origin
@@ -17,17 +20,22 @@
   <joint name="fixed3" type="fixed">
     <origin
+      xyz="0.037646 0.0 0.355"
+      rpy="0 0 3.1415926" />
+    <!--0.037646-->
+    <!--<origin
       xyz="0 0 0.562"
-      rpy="0 0 0" />
-    <parent link="world"/>
-    <child link="mobile_base"/>
+      rpy="0 0 0" /-->
+    <parent link="mobile_base_footprint"/>
+    <child link="base_link"/>
   </joint>
-  <xacro:single_arm side="r"  parent="Arm_Base_R_Link" child="r_tool_link" toolrot="1.57">
-    <origin xyz="0 -0.016 0" rpy="1.57 1.57 0" />
+  <xacro:mir_100 prefix="mobile_"/>
+  <xacro:single_arm side="r"  parent="slide_right" child="r_tool_link" toolrot="1.57">
+    <origin xyz="0.0 0.1151 0.0" rpy="1.57 3.1415926 3.1415926" />
   </xacro:single_arm>
   <xacro:suction side="r"  parent="r_Link_6">
     <origin xyz="0 -0.016 0" rpy="0 0 -1.57" />
   </xacro:suction>
-  <xacro:single_arm side="l"  parent="Arm_Base_L_Link" child="l_tool_link" toolrot="-1.57">
-    <origin xyz="0 0.016 0" rpy="-1.57 1.57 0" />
+  <xacro:single_arm side="l"  parent="slide_left" child="l_tool_link" toolrot="-1.57">
+    <origin xyz="0.0 0.1151 0.0" rpy="-1.57 0 0" />
   </xacro:single_arm>
   <xacro:suction side="l"  parent="l_Link_6">
@@ -41,5 +49,5 @@
     <child link="Base"/>
   </joint-->
-  <joint name="fixed1" type="fixed">
+  <!--<joint name="fixed1" type="fixed">
     <origin
       xyz="0 0 0"
@@ -47,5 +55,5 @@
     <parent link="mobile_base"/>
     <child link="base_link"/>
-  </joint>
+  </joint>-->
   <!--joint name="fixed2" type="fixed">
     <origin
@@ -55,4 +63,5 @@
     <child link="Arm_Base_R"/>
   </joint-->
+<!--
   <link name="Bin">
     <inertial>
@@ -103,7 +112,8 @@
     <child link="Bin"/>
   </joint>
-  <transmission name="tran1_slide_R">
+-->
+  <!-- <transmission name="tran1_slide_R">
     <type>transmission_interface/SimpleTransmission</type>
-    <joint name="slide_R">
+    <joint name="joint_right">
       <hardwareInterface>hardware_interface/PositionJointInterface</hardwareInterface>
     </joint>
@@ -115,5 +125,5 @@
   <transmission name="tran_slide_L">
     <type>transmission_interface/SimpleTransmission</type>
-    <joint name="slide_L">
+    <joint name="joint_left">
       <hardwareInterface>hardware_interface/PositionJointInterface</hardwareInterface>
     </joint>
@@ -122,4 +132,4 @@
       <mechanicalReduction>1</mechanicalReduction>
     </actuator>
-  </transmission>
+  </transmission> -->
 </robot>

File: wrs_gazebo/single_arm/single_arm_description/urdf/single_arm.gazebo.xacro (robot description, xacro)
@@ -6,4 +6,5 @@
       <robotNamespace>/urdf_0129</robotNamespace>
       <robotSimType>gazebo_ros_control/DefaultRobotHWSim</robotSimType>
+      <legacyModeNS>true</legacyModeNS>
     </plugin>
   </gazebo-->
@@ -53,4 +54,25 @@
     <material>Gazebo/Orange</material>
     <selfCollide>false</selfCollide>
+  </gazebo>
+  <gazebo reference="${side}_joint_1">
+    <implicitSpringDamper>True</implicitSpringDamper>
+  </gazebo>
+  <gazebo reference="${side}_joint_2">
+    <implicitSpringDamper>True</implicitSpringDamper>
+  </gazebo>
+  <gazebo reference="${side}_joint_3">
+    <implicitSpringDamper>True</implicitSpringDamper>
+  </gazebo>
+  <gazebo reference="${side}_joint_4">
+    <implicitSpringDamper>True</implicitSpringDamper>
+  </gazebo>
+  <gazebo reference="${side}_joint_5">
+    <implicitSpringDamper>True</implicitSpringDamper>
+  </gazebo>
+  <gazebo reference="${side}_joint_6">
+    <implicitSpringDamper>True</implicitSpringDamper>
+  </gazebo>
+  <gazebo reference="${side}_joint_7">
+    <implicitSpringDamper>True</implicitSpringDamper>
   </gazebo>
   <!-- <gazebo reference="${side}_Link_7">

File: wrs_gazebo/single_arm/single_arm_description/urdf/single_arm.transmission.xacro (robot description, xacro)
@@ -5,8 +5,8 @@
     <type>transmission_interface/SimpleTransmission</type>
     <joint name="${side}_joint_1">
-      <hardwareInterface>hardware_interface/PositionJointInterface</hardwareInterface>
+      <hardwareInterface>hardware_interface/EffortJointInterface</hardwareInterface>
     </joint>
     <actuator name="${side}_motor1">
-      <hardwareInterface>hardware_interface/PositionJointInterface</hardwareInterface>
+      <hardwareInterface>hardware_interface/EffortJointInterface</hardwareInterface>
       <mechanicalReduction>1</mechanicalReduction>
     </actuator>
@@ -15,8 +15,8 @@
     <type>transmission_interface/SimpleTransmission</type>
     <joint name="${side}_joint_2">
-      <hardwareInterface>hardware_interface/PositionJointInterface</hardwareInterface>
+      <hardwareInterface>hardware_interface/EffortJointInterface</hardwareInterface>
     </joint>
     <actuator name="${side}_motor2">
-      <hardwareInterface>hardware_interface/PositionJointInterface</hardwareInterface>
+      <hardwareInterface>hardware_interface/EffortJointInterface</hardwareInterface>
       <mechanicalReduction>1</mechanicalReduction>
     </actuator>
@@ -25,8 +25,8 @@
     <type>transmission_interface/SimpleTransmission</type>
     <joint name="${side}_joint_3">
-      <hardwareInterface>hardware_interface/PositionJointInterface</hardwareInterface>
+      <hardwareInterface>hardware_interface/EffortJointInterface</hardwareInterface>
     </joint>
     <actuator name="${side}_motor3">
-      <hardwareInterface>hardware_interface/PositionJointInterface</hardwareInterface>
+      <hardwareInterface>hardware_interface/EffortJointInterface</hardwareInterface>
       <mechanicalReduction>1</mechanicalReduction>
     </actuator>
@@ -35,8 +35,8 @@
     <type>transmission_interface/SimpleTransmission</type>
     <joint name="${side}_joint_4">
-      <hardwareInterface>hardware_interface/PositionJointInterface</hardwareInterface>
+      <hardwareInterface>hardware_interface/EffortJointInterface</hardwareInterface>
     </joint>
     <actuator name="${side}_motor4">
-      <hardwareInterface>hardware_interface/PositionJointInterface</hardwareInterface>
+      <hardwareInterface>hardware_interface/EffortJointInterface</hardwareInterface>
       <mechanicalReduction>1</mechanicalReduction>
     </actuator>
@@ -45,8 +45,8 @@
     <type>transmission_interface/SimpleTransmission</type>
     <joint name="${side}_joint_5">
-      <hardwareInterface>hardware_interface/PositionJointInterface</hardwareInterface>
+      <hardwareInterface>hardware_interface/EffortJointInterface</hardwareInterface>
     </joint>
     <actuator name="${side}_motor5">
-      <hardwareInterface>hardware_interface/PositionJointInterface</hardwareInterface>
+      <hardwareInterface>hardware_interface/EffortJointInterface</hardwareInterface>
       <mechanicalReduction>1</mechanicalReduction>
     </actuator>
@@ -55,8 +55,8 @@
     <type>transmission_interface/SimpleTransmission</type>
     <joint name="${side}_joint_6">
-      <hardwareInterface>hardware_interface/PositionJointInterface</hardwareInterface>
+      <hardwareInterface>hardware_interface/EffortJointInterface</hardwareInterface>
     </joint>
     <actuator name="${side}_motor6">
-      <hardwareInterface>hardware_interface/PositionJointInterface</hardwareInterface>
+      <hardwareInterface>hardware_interface/EffortJointInterface</hardwareInterface>
       <mechanicalReduction>1</mechanicalReduction>
     </actuator>
@@ -65,8 +65,8 @@
     <type>transmission_interface/SimpleTransmission</type>
     <joint name="${side}_joint_7">
-      <hardwareInterface>hardware_interface/PositionJointInterface</hardwareInterface>
+      <hardwareInterface>hardware_interface/EffortJointInterface</hardwareInterface>
     </joint>
     <actuator name="${side}_motor7">
-      <hardwareInterface>hardware_interface/PositionJointInterface</hardwareInterface>
+      <hardwareInterface>hardware_interface/EffortJointInterface</hardwareInterface>
       <mechanicalReduction>1</mechanicalReduction>
     </actuator>

File: wrs_gazebo/single_arm/single_arm_description/urdf/single_arm.xacro (robot description, xacro)
@@ -10,15 +10,11 @@
 	    <inertial>
 	      <origin
-		xyz="4.11470055452497E-06 -0.000230371464482181 0.0621924893349088"
+		xyz="0.000156250860732315 0.000202963757501797 -0.0546720420122521"
 		rpy="0 0 0" />
 	      <mass
 		value="1.323603974032196" />
-	      <inertia
-		ixx="0.001455064048603135"
-		ixy="-3.55501513691674E-10"
-		ixz="7.08270540818938E-08"
-		iyy="0.001455465136904512"
-		iyz="-4.18207256663005E-06"
-		izz="0.001143220234175012" />
+	      <inertia ixx="0.0001" ixy="0.000"  ixz="0.000"
+         iyy="0.0001" iyz="0.000"
+         izz="0.0001" />
 	    </inertial>
 	    <visual>
@@ -55,15 +51,11 @@
 	    <inertial>
 	      <origin
-		xyz="0.000398625697734733 -3.44839622274201E-06 0.157268979305323"
+		xyz="-3.64540734812575E-06 0.00119778550610652 -0.000421399675048756"
 		rpy="0 0 0" />
 	      <mass
 		value="1.386131223153925" />
-	      <inertia
-		ixx="0.001200765323548107"
-		ixy="6.33822973856499E-08"
-		ixz="3.37474284646834E-06"
-		iyy="0.001623834801578886"
-		iyz="3.68525728102142E-09"
-		izz="0.001612483984092004" />
+	      <inertia ixx="0.0001" ixy="0.000"  ixz="0.000"
+         iyy="0.0001" iyz="0.000"
+         izz="0.0001" />
 	    </inertial>
 	    <visual>
@@ -95,41 +87,93 @@
 	    type="revolute">
 	    <origin
+	      xyz="0 0 0.0550000000000002"
+	      rpy="-1.5707963267949 -2.60398896659329E-32 1.5707963267949" />
+	    <parent
+	      link="${side}_Base" />
+	    <child
+	      link="${side}_Link_1" />
+	    <axis
+	      xyz="0 -1 0" />
+	    <limit
+	      lower="-3.14"
+	      upper="3.14"
+	      effort="1000"
+          velocity="6.5" />
+        <dynamics damping="0.7"/>
+	  </joint>
+	  <link
+	    name="${side}_Link_2">
+	    <inertial>
+	      <origin
+		xyz="0.000683310419598862 -8.00535195483731E-05 0.117541995924546"
+		rpy="0 0 0" />
+	      <mass
+		value="1.479430893999342" />
+	      <inertia ixx="0.0001" ixy="0.000"  ixz="0.000"
+         iyy="0.0001" iyz="0.000"
+         izz="0.0001" />
+	    </inertial>
+	    <visual>
+	      <origin
+		xyz="0 0 0"
+		rpy="0 0 0" />
+	      <geometry>
+		<mesh
+		  filename="package://single_arm_description/meshes/Link_2.STL" />
+	      </geometry>
+	      <material
+		name="">
+		<color
+		  rgba="0.898039215686275 0.917647058823529 0.929411764705882 1" />
+	      </material>
+	    </visual>
+	    <collision>
+	      <origin
+		xyz="0 0 0"
+		rpy="0 0 0" />
+	      <geometry>
+		<mesh
+		  filename="package://single_arm_description/meshes/Link_2.STL" />
+	      </geometry>
+	    </collision>
+	  </link>
+	  <joint
+	    name="${side}_joint_2"
+	    type="revolute">
+	    <origin
 	      xyz="0 0 0"
-	      rpy="0 0 -1.5708" />
-	    <parent
-	      link="${side}_Base" />
-	    <child
+	      rpy="-1.5707963267949 7.39557098644699E-32 -1.5707963267949" />
+	    <parent
 	      link="${side}_Link_1" />
-	    <axis
-	      xyz="0 0 1" />
-	    <limit
-	      lower="-3.14"
-	      upper="3.14"
-	      effort="75"
-	      velocity="65" />
-	  </joint>
-	  <link
-	    name="${side}_Link_2">
-	    <inertial>
-	      <origin
-		xyz="0.0872199190349209 -2.17078867403853E-06 -0.00123755630277769"
-		rpy="0 0 0" />
-	      <mass
-		value="1.479430893999342" />
-	      <inertia
-		ixx="0.002887413979825882"
-		ixy="1.36773393697294E-07"
-		ixz="-4.84905913809873E-05"
-		iyy="0.00222472742020732"
-		iyz="1.07962478497798E-09"
-		izz="0.00177858011962364" />
-	    </inertial>
-	    <visual>
-	      <origin
-		xyz="0 0 0"
-		rpy="0 0 0" />
-	      <geometry>
-		<mesh
-		  filename="package://single_arm_description/meshes/Link_2.STL" />
+	    <child
+	      link="${side}_Link_2" />
+	    <axis
+	      xyz="0 -1 0" />
+	    <limit
+	      lower="-3.14"
+	      upper="3.14"
+	      effort="1000"
+          velocity="6.5" />
+        <dynamics damping="0.7"/>
+	  </joint>
+	  <link
+	    name="${side}_Link_3">
+	    <inertial>
+	      <origin
+		xyz="-0.0220564838621471 0.101455973505417 -8.62457453022769E-05"
+		rpy="0 0 0" />
+	      <mass
+		value="1.568306813792926" />
+	      <inertia ixx="0.0001" ixy="0.000"  ixz="0.000"
+         iyy="0.0001" iyz="0.000"
+         izz="0.0001" />
+	    </inertial>
+	    <visual>
+	      <origin
+		xyz="0 0 0"
+		rpy="0 0 0" />
+	      <geometry>
+		<mesh
+		  filename="package://single_arm_description/meshes/Link_3.STL" />
 	      </geometry>
 	      <material
@@ -145,49 +189,46 @@
 	      <geometry>
 		<mesh
-		  filename="package://single_arm_description/meshes/Link_2.STL" />
-	      </geometry>
-	    </collision>
-	  </link>
-	  <joint
-	    name="${side}_joint_2"
-	    type="revolute">
-	    <origin
-	      xyz="0 0 0.16"
-	      rpy="1.5708 0 1.5708" />
-	    <parent
-	      link="${side}_Link_1" />
-	    <child
+		  filename="package://single_arm_description/meshes/Link_3.STL" />
+	      </geometry>
+	    </collision>
+	  </link>
+	  <joint
+	    name="${side}_joint_3"
+	    type="revolute">
+	    <origin
+	      xyz="0 0 0.174"
+	      rpy="1.5707963267949 4.63843178081015E-17 6.91111242388425E-16" />
+	    <parent
 	      link="${side}_Link_2" />
-	    <axis
-	      xyz="0 0 -1" />
-	    <limit
-	      lower="-3.14"
-	      upper="3.14"
-	      effort="75"
-	      velocity="65" />
-	  </joint>
-	  <link
-	    name="${side}_Link_3">
-	    <inertial>
-	      <origin
-		xyz="-0.0149070189110112 5.93125910155643E-05 0.262650975551228"
-		rpy="0 0 0" />
-	      <mass
-		value="1.568306813792926" />
-	      <inertia
-		ixx="0.000977671503849515"
-		ixy="-1.85851004793169E-06"
-		ixz="0.000224814563369834"
-		iyy="0.000907409589152346"
-		iyz="1.44538660942772E-06"
-		izz="0.000609688957329931" />
-	    </inertial>
-	    <visual>
-	      <origin
-		xyz="0 0 0"
-		rpy="0 0 0" />
-	      <geometry>
-		<mesh
-		  filename="package://single_arm_description/meshes/Link_3.STL" />
+	    <child
+	      link="${side}_Link_3" />
+	    <axis
+	      xyz="0 1 0" />
+	    <limit
+	      lower="-3.14"
+	      upper="3.14"
+	      effort="1000"
+          velocity="6.5" />
+        <dynamics damping="0.7"/>
+	  </joint>
+	  <link
+	    name="${side}_Link_4">
+	    <inertial>
+	      <origin
+		xyz="0.0297389855299131 0.0361651889050357 0.108377256276242"
+		rpy="0 0 0" />
+	      <mass
+		value="1.457613402476782" />
+	      <inertia ixx="0.0001" ixy="0.000"  ixz="0.000"
+         iyy="0.0001" iyz="0.000"
+         izz="0.0001" />
+	    </inertial>
+	    <visual>
+	      <origin
+		xyz="0 0 0"
+		rpy="0 0 0" />
+	      <geometry>
+		<mesh
+		  filename="package://single_arm_description/meshes/Link_4.STL" />
 	      </geometry>
 	      <material
@@ -203,49 +244,101 @@
 	      <geometry>
 		<mesh
-		  filename="package://single_arm_description/meshes/Link_3.STL" />
-	      </geometry>
-	    </collision>
-	  </link>
-	  <joint
-	    name="${side}_joint_3"
-	    type="revolute">
-	    <origin
-	      xyz="0 0 0"
-	      rpy="1.5708 0 1.5708" />
-	    <parent
-	      link="${side}_Link_2" />
-	    <child
+		  filename="package://single_arm_description/meshes/Link_4.STL" />
+	      </geometry>
+	    </collision>
+	  </link>
+	  <joint
+	    name="${side}_joint_4"
+	    type="revolute">
+	    <origin
+	      xyz="-0.0299999998727122 0.115999993001519 0.0359999999999999"
+	      rpy="-1.5707963267949 -1.40443212615082E-14 1.75438367537121E-15" />
+	    <parent
 	      link="${side}_Link_3" />
-	    <axis
-	      xyz="0 0 1" />
-	    <limit
-	      lower="-3.14"
-	      upper="3.14"
-	      effort="65"
-	      velocity="65" />
-	  </joint>
-	  <link
-	    name="${side}_Link_4">
-	    <inertial>
-	      <origin
-		xyz="-0.0294457805062883 -0.0888739607940883 8.91006395364796E-05"
-		rpy="0 0 0" />
-	      <mass
-		value="1.457613402476782" />
-	      <inertia
-		ixx="0.00203111007559186"
-		ixy="-3.51922856144699E-05"
-		ixz="1.00599592333376E-06"
-		iyy="0.000727015941977056"
-		iyz="-1.55525051076035E-07"
-		izz="0.0017620916887768" />
-	    </inertial>
-	    <visual>
-	      <origin
-		xyz="0 0 0"
-		rpy="0 0 0" />
-	      <geometry>
-		<mesh
-		  filename="package://single_arm_description/meshes/Link_4.STL" />
+	    <child
+	      link="${side}_Link_4" />
+	    <axis
+	      xyz="0 -1 0" />
+	    <limit
+	      lower="-3.14"
+	      upper="3.14"
+	      effort="1000"
+          velocity="6.5" />
+        <dynamics damping="0.7"/>
+	  </joint>
+	  <link
+	    name="${side}_Link_5">
+	    <inertial>
+	      <origin
+		xyz="-0.000172095429412281 0.102690028206534 -6.66794215013755E-05"
+		rpy="0 0 0" />
+	      <mass
+		value="1.448277275798768" />
+	      <inertia ixx="0.0001" ixy="0.000"  ixz="0.000"
+         iyy="0.0001" iyz="0.000"
+         izz="0.0001" />
+	    </inertial>
+	    <visual>
+	      <origin
+		xyz="0 0 0"
+		rpy="0 0 0" />
+	      <geometry>
+		<mesh
+		  filename="package://single_arm_description/meshes/Link_5.STL" />
+	      </geometry>
+	      <material
+		name="">
+		<color
+		  rgba="0.792156862745098 0.819607843137255 0.933333333333333 1" />
+	      </material>
+	    </visual>
+	    <collision>
+	      <origin
+		xyz="0 0 0"
+		rpy="0 0 0" />
+	      <geometry>
+		<mesh
+		  filename="package://single_arm_description/meshes/Link_5.STL" />
+	      </geometry>
+	    </collision>
+	  </link>
+	  <joint
+	    name="${side}_joint_5"
+	    type="revolute">
+	    <origin
+	      xyz="0.029999999872713 0.0359999999999987 0.162"
+	      rpy="1.5707963267949 -8.80083043478898E-16 -2.49800180540655E-16" />
+	    <parent
+	      link="${side}_Link_4" />
+	    <child
+	      link="${side}_Link_5" />
+	    <axis
+	      xyz="0 1 0" />
+	    <limit
+	      lower="-3.14"
+	      upper="3.14"
+	      effort="1000"
+          velocity="6.5" />
+        <dynamics damping="0.7"/>
+	  </joint>
+	  <link
+	    name="${side}_Link_6">
+	    <inertial>
+	      <origin
+		xyz="1.14707347786958E-08 0.0359051244401507 0.076720238383497"
+		rpy="0 0 0" />
+	      <mass
+		value="1.205818407044008" />
+	      <inertia ixx="0.0001" ixy="0.000"  ixz="0.000"
+         iyy="0.0001" iyz="0.000"
+         izz="0.0001" />
+	    </inertial>
+	    <visual>
+	      <origin
+		xyz="0 0 0"
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
File: wrs_gazebo/slide_rail/urdf/slide_rail.xacro (robot description, xacro)
@@ -43,5 +43,5 @@
   </link>
   <link
-    name="Arm_Base_R_Link">
+    name="slide_right">
     <inertial>
       <origin
@@ -83,5 +83,5 @@
   </link>
   <joint
-    name="slide_R"
+    name="joint_right"
     type="prismatic">
     <origin
@@ -91,5 +91,5 @@
       link="base_link" />
     <child
-      link="Arm_Base_R_Link" />
+      link="slide_right" />
     <axis
       xyz="0 0 1" />
@@ -101,5 +101,5 @@
   </joint>
   <link
-    name="Arm_Base_L_Link">
+    name="slide_left">
     <inertial>
       <origin
@@ -141,5 +141,5 @@
   </link>
   <joint
-    name="slide_L"
+    name="joint_left"
     type="prismatic">
     <origin
@@ -149,5 +149,5 @@
       link="base_link" />
     <child
-      link="Arm_Base_L_Link" />
+      link="slide_left" />
     <axis
       xyz="0 0 1" />
@@ -158,25 +158,23 @@
       velocity="100" />
   </joint>
-<!--
-  <transmission name="tran1">
+  <transmission name="slide_tran_r">
     <type>transmission_interface/SimpleTransmission</type>
-    <joint name="slide_R">
-      <hardwareInterface>hardware_interface/PositionJointInterface</hardwareInterface>
+    <joint name="joint_right">
+      <hardwareInterface>hardware_interface/EffortJointInterface</hardwareInterface>
     </joint>
-    <actuator name="motor1">
-      <hardwareInterface>hardware_interface/PositionJointInterface</hardwareInterface>
+    <actuator name="slide_motor_r">
+      <hardwareInterface>hardware_interface/EffortJointInterface</hardwareInterface>
       <mechanicalReduction>1</mechanicalReduction>
     </actuator>
   </transmission>
-  <transmission name="tran2">
+  <transmission name="slide_tran_l">
     <type>transmission_interface/SimpleTransmission</type>
-    <joint name="slide_L">
-      <hardwareInterface>hardware_interface/PositionJointInterface</hardwareInterface>
+    <joint name="joint_left">
+      <hardwareInterface>hardware_interface/EffortJointInterface</hardwareInterface>
     </joint>
-    <actuator name="motor2">
-      <hardwareInterface>hardware_interface/PositionJointInterface</hardwareInterface>
+    <actuator name="slide_motor_l">
+      <hardwareInterface>hardware_interface/EffortJointInterface</hardwareInterface>
       <mechanicalReduction>1</mechanicalReduction>
     </actuator>
   </transmission>
--->
 </robot>

File: wrs_gazebo/suction_urdf/urdf/suction.transmission.xacro (robot description, xacro)
@@ -5,8 +5,8 @@
     <type>transmission_interface/SimpleTransmission</type>
     <joint name="${side}_tool_joint">
-      <hardwareInterface>hardware_interface/PositionJointInterface</hardwareInterface>
+      <hardwareInterface>hardware_interface/EffortJointInterface</hardwareInterface>
     </joint>
     <actuator name="${side}_suction_motor1">
-      <hardwareInterface>hardware_interface/PositionJointInterface</hardwareInterface>
+      <hardwareInterface>hardware_interface/EffortJointInterface</hardwareInterface>
       <mechanicalReduction>1</mechanicalReduction>
     </actuator>
