Commit message: Add Mir into Gazebo, Files not been Organized

File: wrs_gazebo/suction_urdf/urdf/suction_urdf.xacro (robot description, xacro)
@@ -12,11 +12,7 @@
         <mass
           value="0.11123" />
-        <inertia
-          ixx="8.4875E-05"
-          ixy="4.1003E-07"
-          ixz="4.0241E-06"
-          iyy="0.00010438"
-          iyz="6.5325E-07"
-          izz="4.7593E-05" />
+        <inertia ixx="0.0001" ixy="0.000"  ixz="0.000"
+         iyy="0.0001" iyz="0.000"
+         izz="0.0001" />
       </inertial>
       <visual>
@@ -52,11 +48,7 @@
         <mass
           value="0.033438" />
-        <inertia
-          ixx="2.0813E-05"
-          ixy="1.7379E-08"
-          ixz="9.2823E-08"
-          iyy="1.8619E-05"
-          iyz="4.6462E-06"
-          izz="5.6779E-06" />
+        <inertia ixx="0.0001" ixy="0.000"  ixz="0.000"
+         iyy="0.0001" iyz="0.000"
+         izz="0.0001" />
       </inertial>
       <visual>
@@ -98,7 +90,8 @@
       <limit
         lower="-3.14"
-	      upper="3.14"
-        effort="5"
-        velocity="0.5" />
+	    upper="3.14"
+        effort="1000"
+        velocity="6.5" />
+      <dynamics damping="0.7"/>
     </joint>
     <link
@@ -111,11 +104,7 @@
         <mass
           value="0.0001" />
-        <inertia
-          ixx="2.0813E-05"
-          ixy="1.7379E-08"
-          ixz="9.2823E-08"
-          iyy="1.8619E-05"
-          iyz="4.6462E-06"
-          izz="5.6779E-06" />
+        <inertia ixx="0.0001" ixy="0.000"  ixz="0.000"
+         iyy="0.0001" iyz="0.000"
+         izz="0.0001" />
       </inertial>
       <visual>
@@ -144,6 +133,6 @@
             lower="0"
 	    upper="0"
-            effort="5"
-            velocity="5" />
+            effort="1000"
+            velocity="6.5" />
         <dynamics damping="0.0" friction="10"/>
     </joint>
@@ -157,11 +146,7 @@
         <mass
           value="0.0001" />
-        <inertia
-          ixx="2.0813E-05"
-          ixy="1.7379E-08"
-          ixz="9.2823E-08"
-          iyy="1.8619E-05"
-          iyz="4.6462E-06"
-          izz="5.6779E-06" />
+        <inertia ixx="0.0001" ixy="0.000"  ixz="0.000"
+         iyy="0.0001" iyz="0.000"
+         izz="0.0001" />
       </inertial>
       <visual>
@@ -190,6 +175,6 @@
             lower="0"
 	    upper="0"
-            effort="5"
-            velocity="5" />
+            effort="1000"
+            velocity="6.5" />
         <dynamics damping="0.0" friction="10"/>
     </joint>
@@ -203,11 +188,7 @@
         <mass
           value="0.0001" />
-        <inertia
-          ixx="2.0813E-05"
-          ixy="1.7379E-08"
-          ixz="9.2823E-08"
-          iyy="1.8619E-05"
-          iyz="4.6462E-06"
-          izz="5.6779E-06" />
+        <inertia ixx="0.0001" ixy="0.000"  ixz="0.000"
+         iyy="0.0001" iyz="0.000"
+         izz="0.0001" />
       </inertial>
       <visual>
@@ -236,6 +217,6 @@
             lower="0"
 	    upper="0"
-            effort="5"
-            velocity="5" />
+            effort="1000"
+            velocity="6.5" />
         <dynamics damping="0.0" friction="10"/>
     </joint>
@@ -249,11 +230,7 @@
         <mass
           value="0.0001" />
-        <inertia
-          ixx="2.0813E-05"
-          ixy="1.7379E-08"
-          ixz="9.2823E-08"
-          iyy="1.8619E-05"
-          iyz="4.6462E-06"
-          izz="5.6779E-06" />
+        <inertia ixx="0.0001" ixy="0.000"  ixz="0.000"
+         iyy="0.0001" iyz="0.000"
+         izz="0.0001" />
       </inertial>
       <visual>
@@ -282,6 +259,6 @@
             lower="0"
 	    upper="0"
-            effort="5"
-            velocity="5" />
+            effort="1000"
+            velocity="6.5" />
         <dynamics damping="0.0" friction="10"/>
     </joint>
@@ -295,11 +272,7 @@
         <mass
           value="0.0001" />
-        <inertia
-          ixx="2.0813E-05"
-          ixy="1.7379E-08"
-          ixz="9.2823E-08"
-          iyy="1.8619E-05"
-          iyz="4.6462E-06"
-          izz="5.6779E-06" />
+        <inertia ixx="0.0001" ixy="0.000"  ixz="0.000"
+         iyy="0.0001" iyz="0.000"
+         izz="0.0001" />
       </inertial>
       <visual>
@@ -327,7 +300,7 @@
         <limit
             lower="0"
-	    upper="0"
-            effort="5"
-            velocity="5" />
+	        upper="0"
+            effort="1000"
+            velocity="6.5" />
         <dynamics damping="0.0" friction="10"/>
     </joint>

Commit message: Edit Stocking Task

File: wrs_gazebo/mobile_dual_arm/urdf/mobile_dual_arm.xacro (robot description, xacro)
@@ -30,5 +30,5 @@
   </joint>
   <xacro:mir_100 prefix="mobile_"/>
-  <xacro:single_arm side="r"  parent="slide_right" child="r_tool_link" toolrot="1.57">
+  <xacro:single_arm side="r"  parent="slide_right" child="r_tool_link" toolrot="-1.57">
     <origin xyz="0.0 0.1151 0.0" rpy="1.57 3.1415926 3.1415926" />
   </xacro:single_arm>
@@ -36,5 +36,5 @@
     <origin xyz="0 -0.016 0" rpy="0 0 -1.57" />
   </xacro:suction>
-  <xacro:single_arm side="l"  parent="slide_left" child="l_tool_link" toolrot="-1.57">
+  <xacro:single_arm side="l"  parent="slide_left" child="l_tool_link" toolrot="1.57">
     <origin xyz="0.0 0.1151 0.0" rpy="-1.57 0 0" />
   </xacro:single_arm>
@@ -63,43 +63,42 @@
     <child link="Arm_Base_R"/>
   </joint-->
-<!--
   <link name="Bin">
     <inertial>
       <origin
-	xyz="0 0 0"
-	rpy="0 0 0" />
+      	xyz="0 0 0"
+      	rpy="0 0 0" />
       <mass
-	value="0.823603974032196" />
+      	value="0.823603974032196" />
       <inertia
-	ixx="0"
-	ixy="0"
-	ixz="0"
-	iyy="0"
-	iyz="0"
-	izz="0" />
+      	ixx="1"
+      	ixy="0"
+      	ixz="0"
+      	iyy="1"
+      	iyz="0"
+      	izz="1" />
     </inertial>
     <visual>
       <origin
-	xyz="0 0 0"
-	rpy="0 0 0" />
+      	xyz="0 0 0"
+      	rpy="0 0 0" />
       <geometry>
-	<mesh
-          scale="0.001 0.001 0.001"
-	  filename="package://mobile_dual_arm/scene/meshes/bin.STL" />
+	    <mesh
+        scale="0.001 0.001 0.001"
+	      filename="package://mobile_dual_arm/scene/meshes/bin.STL" />
       </geometry>
       <material
-	name="blue_">
-	<color
-	  rgba="0.4 0.66 0.99 1" />
+      	name="blue_">
+       	<color
+       	  rgba="0.4 0.66 0.99 1" />
       </material>
     </visual>
     <collision>
       <origin
-	xyz="0 0 0"
-	rpy="0 0 0" />
+	      xyz="0 0 0"
+      	rpy="0 0 0" />
       <geometry>
-	<mesh
+      	<mesh
           scale="0.001 0.001 0.001"
-	  filename="package://mobile_dual_arm/scene/meshes/bin.STL" />
+	        filename="package://mobile_dual_arm/scene/meshes/bin.STL" />
       </geometry>
     </collision>
@@ -107,29 +106,8 @@
   <joint name="fixed4" type="fixed">
     <origin
-      xyz="-0.175 -0.31 0.06"
+      xyz="0.35 -0.31 0.26"
       rpy="0 0 1.5708" />
-    <parent link="mobile_base"/>
+    <parent link="base_link"/>
     <child link="Bin"/>
   </joint>
--->
-  <!-- <transmission name="tran1_slide_R">
-    <type>transmission_interface/SimpleTransmission</type>
-    <joint name="joint_right">
-      <hardwareInterface>hardware_interface/PositionJointInterface</hardwareInterface>
-    </joint>
-    <actuator name="motor1_slide_R">
-      <hardwareInterface>hardware_interface/PositionJointInterface</hardwareInterface>
-      <mechanicalReduction>1</mechanicalReduction>
-    </actuator>
-  </transmission>
-  <transmission name="tran_slide_L">
-    <type>transmission_interface/SimpleTransmission</type>
-    <joint name="joint_left">
-      <hardwareInterface>hardware_interface/PositionJointInterface</hardwareInterface>
-    </joint>
-    <actuator name="motor_slide_L">
-      <hardwareInterface>hardware_interface/PositionJointInterface</hardwareInterface>
-      <mechanicalReduction>1</mechanicalReduction>
-    </actuator>
-  </transmission> -->
 </robot>

File: wrs_gazebo/single_arm/single_arm_description/urdf/single_arm.xacro (robot description, xacro)
@@ -14,7 +14,7 @@
 	      <mass
 		value="0.323603974032196" />
-	      <inertia ixx="0.0001" ixy="0.000"  ixz="0.000"
-         iyy="0.0001" iyz="0.000"
-         izz="0.0001" />
+	      <inertia ixx="0.1" ixy="0.0"  ixz="0.0"
+         iyy="0.1" iyz="0.0"
+         izz="0.1" />
 	    </inertial>
 	    <visual>
@@ -55,7 +55,7 @@
 	      <mass
 		value="0.386131223153925" />
-	      <inertia ixx="0.0001" ixy="0.000"  ixz="0.000"
-         iyy="0.0001" iyz="0.000"
-         izz="0.0001" />
+	      <inertia ixx="0.1" ixy="0.0"  ixz="0.0"
+         iyy="0.1" iyz="0.0"
+         izz="0.1" />
 	    </inertial>
 	    <visual>
@@ -110,7 +110,7 @@
 	      <mass
 		value="0.479430893999342" />
-	      <inertia ixx="0.0001" ixy="0.000"  ixz="0.000"
-         iyy="0.0001" iyz="0.000"
-         izz="0.0001" />
+	      <inertia ixx="0.1" ixy="0.0"  ixz="0.0"
+         iyy="0.1" iyz="0.0"
+         izz="0.1" />
 	    </inertial>
 	    <visual>
@@ -165,7 +165,7 @@
 	      <mass
 		value="0.568306813792926" />
-	      <inertia ixx="0.0001" ixy="0.000"  ixz="0.000"
-         iyy="0.0001" iyz="0.000"
-         izz="0.0001" />
+	      <inertia ixx="0.1" ixy="0.0"  ixz="0.0"
+         iyy="0.1" iyz="0.0"
+         izz="0.1" />
 	    </inertial>
 	    <visual>
@@ -220,7 +220,7 @@
 	      <mass
 		value="0.457613402476782" />
-	      <inertia ixx="0.0001" ixy="0.000"  ixz="0.000"
-         iyy="0.0001" iyz="0.000"
-         izz="0.0001" />
+	      <inertia ixx="0.1" ixy="0.0"  ixz="0.0"
+         iyy="0.1" iyz="0.0"
+         izz="0.1" />
 	    </inertial>
 	    <visual>
@@ -275,7 +275,7 @@
 	      <mass
 		value="0.448277275798768" />
-	      <inertia ixx="0.0001" ixy="0.000"  ixz="0.000"
-         iyy="0.0001" iyz="0.000"
-         izz="0.0001" />
+	      <inertia ixx="0.1" ixy="0.0"  ixz="0.0"
+         iyy="0.1" iyz="0.0"
+         izz="0.1" />
 	    </inertial>
 	    <visual>
@@ -330,7 +330,7 @@
 	      <mass
 		value="0.205818407044008" />
-	      <inertia ixx="0.0001" ixy="0.000"  ixz="0.000"
-         iyy="0.0001" iyz="0.000"
-         izz="0.0001" />
+	      <inertia ixx="0.1" ixy="0.0"  ixz="0.0"
+         iyy="0.1" iyz="0.0"
+         izz="0.1" />
 	    </inertial>
 	    <visual>
@@ -422,5 +422,5 @@
 			<origin
 				xyz="0 0.03680 0.135"
-				rpy="0 0 0" />
+				rpy="0 0 ${toolrot}" />
 				<!-- rpy="1.5708 ${toolrot} 0" /> -->
 				<!-- xyz="-0.008041 0.038 0.13545" -->

File: wrs_gazebo/suction_urdf/urdf/suction_urdf.xacro (robot description, xacro)
@@ -12,8 +12,8 @@
         <mass
           value="0.11123" />
-        <inertia ixx="0.0001" ixy="0.000"  ixz="0.000"
-         iyy="0.0001" iyz="0.000"
-         izz="0.0001" />
-      </inertial>
+        <inertia ixx="0.1" ixy="0.0"  ixz="0.0"
+         iyy="0.1" iyz="0.0"
+         izz="0.1" />
+	    </inertial>
       <visual>
         <origin
@@ -48,8 +48,8 @@
         <mass
           value="0.033438" />
-        <inertia ixx="0.0001" ixy="0.000"  ixz="0.000"
-         iyy="0.0001" iyz="0.000"
-         izz="0.0001" />
-      </inertial>
+        <inertia ixx="0.1" ixy="0.0"  ixz="0.0"
+         iyy="0.1" iyz="0.0"
+         izz="0.1" />
+	    </inertial>
       <visual>
         <origin

Commit message: Add Relative Movement in GUI

File: wrs_gazebo/mobile_dual_arm/urdf/mobile_dual_arm.xacro (robot description, xacro)
@@ -10,12 +10,12 @@
   <xacro:include filename="$(find mobile_dual_arm)/urdf/mobile_dual_arm.gazebo" />
   <!--xacro:include filename="$(find mobile_table)/urdf/mobile_table.xacro" /-->
-  <!--<link name="world"/-->
-  <!-- <joint name="fixed1" type="fixed">
+  <link name="world"/>
+  <joint name="fixed1" type="fixed">
     <origin
-      xyz="0 0 0.562"
+      xyz="0 0 0"
       rpy="0 0 0" />
     <parent link="world"/>
-    <child link="base_link"/>
-  </joint> -->
+    <child link="mobile_base_footprint"/>
+  </joint>
   <joint name="fixed3" type="fixed">
     <origin
